File: hw/RemoteController/Radio.kicad_sch (KiCad schematic)
At the start: 70 parts, among them J2 BWSMA-KWE-Z3.5*4.2, U1 XA17-G4K, U11 LM358, U12 GVA-63, U13 LM358, U17 AD8314RM, U18 AD8314RM, U2 SPF5043Z, U3 MICRF220AYQS, U4 H3-TCD-12-222X+, U7 H3-TCD-12-222X+, U9 MAX7044AKA, Y1 L327S13CU11L, Y4 13.56 MHz

Commit message: remote_ctrl: last commit before re-routing
Parts:
- C1: PN (none) -> CL05A104KA5NNNC
- C10: renamed from C12; PN (none) -> CL05A475MO5NUNC
- C13: renamed from C15; PN (none) -> TCC0402X7R102K500AT
- C17: renamed from C19; PN (none) -> TCC0402X7R102K500AT
- C18: renamed from C20; PN (none) -> TCC0402X7R102K500AT
- C2: renamed from C5; PN (none) -> CL05A104KA5NNNC
- C20: renamed from C22; PN (none) -> CL05A104KA5NNNC
- C22: renamed from C24; PN (none) -> TCC0402X7R102K500AT
- C25: renamed from C28; PN (none) -> CL05A104KA5NNNC
- C26: renamed from C29; PN (none) -> 0402B221K500NT
- C27: renamed from C30; PN (none) -> CC0402JRNPO9BN681
- C3: renamed from C2; PN (none) -> CL05A104KA5NNNC
- C30: renamed from C33; PN (none) -> CC0402JRNPO9BN681
- C32: renamed from C35; PN (none) -> CC0402JRNPO9BN100
- C33: renamed from C36; PN (none) -> CC0402JRNPO9BN100
- C36: renamed from C40; PN (none) -> CL05A104KA5NNNC
- C37: renamed from C41; PN (none) -> TCC0402X7R102K500AT
- C38: renamed from C42; PN (none) -> CL05A104KA5NNNC
- C39: renamed from C43; PN (none) -> TCC0402X7R102K500AT
- C4: renamed from C6; PN (none) -> CL05A104KA5NNNC
- C40: renamed from C44; PN (none) -> CC0402JRNPO9BN120
- C41: renamed from C45; PN (none) -> CC0402JRNPO9BN180
- C42: renamed from C46; PN (none) -> CC0402JRNPO9BN150
- C43: renamed from C47; PN (none) -> CL05A104KA5NNNC
- C44: renamed from C48; PN (none) -> CC0402JRNPO9BN681
- C45: renamed from C49; PN (none) -> 0402B221K500NT
- C46: renamed from C50; PN (none) -> CL05A104KA5NNNC
- C5: renamed from C7; PN (none) -> CC0402JRNPO9BN681
- C6: renamed from C8; PN (none) -> 0402B221K500NT
- C7: renamed from C9; PN (none) -> CC0402JRNPO9BN100
- C8: renamed from C10; PN (none) -> CC0402JRNPO9BN100
- C9: renamed from C11; PN (none) -> TCC0402X7R102K500AT
- R1: PN (none) -> FRC0402J103 TS
- R11: renamed from R12; PN (none) -> FRC0402J103 TS
- R12: renamed from R13; PN (none) -> RT0402BRE0750RL
- R13: renamed from R39; PN (none) -> FRC0402F52R3TS
- R14: renamed from R25; PN (none) -> CR0402-FX-10R0GLF
- R15: renamed from R14; PN (none) -> RT0402BRD07100RL
- R16: renamed from R15; PN (none) -> RT0402BRE0750RL
- R19: renamed from R20; PN (none) -> FRC0402F91R0TS
- R2: PN (none) -> CR0402-FX-10R0GLF
- R20: renamed from R21; PN (none) -> FRC0402J820 TS
- R22: renamed from R23; PN (none) -> FRC0402F52R3TS
- R23: renamed from R24; PN (none) -> FRC0402F91R0TS
- R24: renamed from R40; PN (none) -> CRCW04020000Z0EE
- R27: renamed from R28; PN (none) -> RT0402BRD07100RL
- R28: renamed from R29; PN (none) -> RT0402BRD07100RL
- R29: renamed from R30; PN (none) -> RT0402BRD07100RL
- R3: renamed from R4; PN (none) -> FRC0402J103 TS
- R30: renamed from R31; PN (none) -> RT0402BRD07100RL
- R7: renamed from R8; PN (none) -> FRC0402J103 TS
- U11, U13: PN (none) -> LM358
- U12: PN (none) -> GVA-63+
- U2: PN (none) -> SPF5043Z
- U3: PN (none) -> MICRF220AYQS-TR
- U4: PN (none) -> H3-TCD-12-222X+
- U6: renamed from U18; PN (none) -> AD8314ARMZ-REEL
- U7: renamed from U17; PN (none) -> AD8314ARMZ-REEL
- U8: renamed from U7; PN (none) -> H3-TCD-12-222X+
- U9: PN (none) -> MAX7044AKA+T
- Y1: PN (none) -> L327S120U11L
