File: hw/RemoteController/RemoteController.kicad_pcb (KiCad board)
At the start: 4 copper layers, 100 x 75 mm, 136 parts, among them J1 Conn_01x04_Pin, J2 BWSMA-KWE-Z3.5*4.2, J5 Conn_01x04_Pin, SW1 ST-0-102-A01-T000-LF, SW2 TS-1088-AR02016, SW3 TS-1088-AR02016, SW4 TS-1088-AR02016, SW5 TS-1088-AR02016, U1 XA17-G4K, U10 LM358, U11 LM358, U12 GVA-63, U13 LM358, U14 LM358, U15 LM358, U16 TPS562200, U17 AD8314RM, U18 AD8314RM, U2 SPF5043Z, U3 MICRF220AYQS, U4 H3-TCD-12-222X+, U5 nRF52810-QFxx, U7 H3-TCD-12-222X+, U9 MAX7044AKA, Y1 L327S13CU11L, Y2 32 MHz, Y3 32.768 KHz, Y4 13.56 MHz

Commit message: remote_ctrl: last commit before re-routing
Parts:
- added J7: Conn_01x01_Pin, Connector_PinSocket_2.54mm:PinSocket_1x01_P2.54mm_Vertical, F.Cu at (133.5, 97.5)
- added J8: Conn_01x01_Pin, Connector_PinSocket_2.54mm:PinSocket_1x01_P2.54mm_Vertical, F.Cu at (157.0, 97.5)
- renumbered C12 to C10, C13 to C11, C14 to C12, C15 to C13, C16 to C14, C17 to C15, C18 to C16, C19 to C17, C20 to C18, C21 to C19, C5 to C2, C22 to C20, C23 to C21, C24 to C22, C25 to C23, C26 to C24, C28 to C25, C29 to C26, C30 to C27, C31 to C28, C32 to C29, C2 to C3, C33 to C30, C34 to C31, C35 to C32, C36 to C33, C37 to C34, C38 to C35, C40 to C36, C41 to C37, C42 to C38, C43 to C39, C6 to C4, C44 to C40, C45 to C41, C46 to C42, C47 to C43, C48 to C44, C49 to C45, C50 to C46, C51 to C47, C52 to C48, C53 to C49, C7 to C5, C54 to C50, C55 to C51, C56 to C52, C57 to C53, C8 to C6, C9 to C7, C10 to C8, C11 to C9, R11 to R10, R12 to R11, R13 to R12, R39 to R13, R25 to R14, R14 to R15, R15 to R16, R20 to R19, R21 to R20, R22 to R21, R23 to R22, R24 to R23, R40 to R24, R26 to R25, R27 to R26, R28 to R27, R29 to R28, R30 to R29, R4 to R3, R31 to R30, R32 to R31, R33 to R32, R34 to R33, R35 to R34, R36 to R35, R37 to R36, R38 to R37, R5 to R4, R6 to R5, R7 to R6, R8 to R7, R9 to R8, R10 to R9, U18 to U6, U17 to U7, U7 to U8
Other:
- board text added: "TEST_GND"
- board text added: "TEST_VIN"
