File: hw/RemoteController/RemoteController.kicad_sch (KiCad schematic)
At the start: 67 parts, among them J1 Conn_01x04_Pin, J5 Conn_01x04_Pin, SW1 ST-0-102-A01-T000-LF, SW2 TS-1088-AR02016, SW3 TS-1088-AR02016, SW4 TS-1088-AR02016, SW5 TS-1088-AR02016, U10 LM358, U13 LM358, U14 LM358, U15 LM358, U16 TPS562200, U5 nRF52810-QFxx, Y2 32 MHz, Y3 32.768 KHz

Commit message: remote_ctrl: last commit before re-routing
Parts:
- added J7, J8: Conn_01x01_Pin, Connector_PinSocket_2.54mm:PinSocket_1x01_P2.54mm_Vertical, symbol Connector:Conn_01x01_Pin
- AE1: PN (none) -> 2450AT18A100E
- BT1, BT2: PN (none) -> BH-AAA-B5BA021
- C11: renamed from C13; PN (none) -> CL05A104KA5NNNC
- C12: renamed from C14; PN (none) -> CL05A105KO5NNNC
- C14: renamed from C16; PN (none) -> CC0402JRNPO9BN200
- C15: renamed from C17; PN (none) -> CC0402JRNPO9BN200
- C16: renamed from C18; PN (none) -> CC0402JRNPO9BN200
- C19: renamed from C21; PN (none) -> CC0402KRX7R8BB101
- C21: renamed from C23; PN (none) -> CC0402JRNPO9BN200
- C23: renamed from C25; PN (none) -> CC0402BRNPO9BN1R0
- C24: renamed from C26; PN (none) -> GJM1555C1H1R2WB01D
- C28: renamed from C31; PN (none) -> CL05A104KA5NNNC
- C29: renamed from C32; PN (none) -> CL05A104KA5NNNC
- C31: renamed from C34; PN (none) -> CL05A475MO5NUNC
- C34: renamed from C37; PN (none) -> CL05A104KA5NNNC
- C35: renamed from C38; PN (none) -> CL05A104KA5NNNC
- C47: renamed from C51; PN (none) -> CL05A104KA5NNNC
- C48: renamed from C52; PN (none) -> CL05A104KA5NNNC
- C49: renamed from C53; PN (none) -> GRM155R60J226ME11D
- C50: renamed from C54; PN (none) -> GRM155R60J226ME11D
- C51: renamed from C55; PN (none) -> CL05A104KA5NNNC
- C52: renamed from C56; PN (none) -> CL05A106MQ5NUNC
- C53: renamed from C57; PN (none) -> CL05A106MQ5NUNC
- J1: now left out of the parts list
- J3, J4: PN (none) -> YG16-FL7.8-B10Ka(80)-R
- L3: PN (none) -> VHF160808H4N7ST
- L4: PN (none) -> CS0603-2N2J-S
- L8: PN (none) -> CMH160808B2R2MT
- R10: renamed from R11; PN (none) -> RT0402BRD071KL
- R17: PN (none) -> RT0402BRD071KL
- R18: PN (none) -> CRCW040250K0FKED
- R21: renamed from R22; PN (none) -> CRCW040250K0FKED
- R25: renamed from R26; PN (none) -> CRCW04020000Z0EE
- R26: renamed from R27; PN (none) -> CRCW04020000Z0EE
- R31: renamed from R32; PN (none) -> FRC0402J103 TS
- R32: renamed from R33; PN (none) -> FRC0402J103 TS
- R33: renamed from R34; PN (none) -> CRCW04020000Z0EE
- R34: renamed from R35; PN (none) -> CRCW040250K0FKED
- R35: renamed from R36; PN (none) -> FRC0402J103 TS
- R36: renamed from R37; PN (none) -> CRCW04023K30FKED
- R37: renamed from R38; PN (none) -> FRC0402F5101TS
- R4: renamed from R5; PN (none) -> CRCW040250K0FKED
- R5: renamed from R6; PN (none) -> CRCW040250K0FKED
- R6: renamed from R7; PN (none) -> CRCW040250K0FKED
- R8: renamed from R9; PN (none) -> RT0402BRD071KL
- R9: renamed from R10; PN (none) -> RT0402BRD071KL
- SW2, SW3, SW4, SW5: PN TC-6610-6*6*8-300g -> TS-1088-AR02016
- U10, U13, U14, U15: PN (none) -> LM358
- U5: PN (none) -> NRF52810-QFAA-T
Connections:
- net GND: now also J8.1 (Pin_1)
- net VBAT2: now also J7.1 (Pin_1)
Other:
- moved on the sheet: BT1, BT2, C34, C35, C49, C50, C51, C52, C53, L8, R25, R26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
